File: cheapino.kicad_sch (KiCad schematic)
At the start: 42 parts, among them K1 SW_Push, K10 SW_Push, K11 SW_Push, K12 SW_Push, K13 SW_Push, K14 SW_Push, K15 SW_Push, K16 SW_Push, K17 SW_Push, K18 SW_Push, K2 SW_Push, K3 SW_Push, K4 SW_Push, K5 SW_Push, K6 SW_Push, K7 SW_Push, K8 SW_Push, K9 SW_Push, U1 RP2040-Zero

Commit message: actually changed pcb
Parts:
- D1, D10, D11, D12, D13, D14, D15, D17, D18, D19, D2, D20, D3, D4, D5, D6, D7, D8, D9: footprint keebio:Diode-dual -> keebio-parts:Diode-dual
- K1, K10, K11, K12, K13, K14, K15, K16, K17, K18, K2, K3, K4, K5, K6, K7, K8, K9: footprint project_footprints:SW_MX_reversible_minimal -> keyswitches:Kailh_socket_MX_optional_reversible
