File: cheapino.kicad_pcb (KiCad board)
At the start: 2 copper layers, 139 x 102.6 mm, 42 parts, among them K1 SW_Push, K10 SW_Push, K11 SW_Push, K12 SW_Push, K13 SW_Push, K14 SW_Push, K15 SW_Push, K16 SW_Push, K17 SW_Push, K18 SW_Push, K2 SW_Push, K3 SW_Push, K4 SW_Push, K5 SW_Push, K6 SW_Push, K7 SW_Push, K8 SW_Push, K9 SW_Push, U1 RP2040-Zero

Commit message: actually changed pcb
Parts:
- added REF**: MountingHole_2.2mm_M2_ISO7380, MountingHole:MountingHole_2.2mm_M2_ISO7380, F.Cu at (131.3, 131.6)
- added REF**: MountingHole_2.2mm_M2_ISO7380, MountingHole:MountingHole_2.2mm_M2_ISO7380, F.Cu at (151.7, 117.4)
- added REF**: MountingHole_2.2mm_M2_ISO7380, MountingHole:MountingHole_2.2mm_M2_ISO7380, F.Cu at (185.7, 141.2)
- added REF**: MountingHole_2.2mm_M2_ISO7380, MountingHole:MountingHole_2.2mm_M2_ISO7380, F.Cu at (60.6, 116.9)
- added REF**: MountingHole_2.2mm_M2_ISO7380, MountingHole:MountingHole_2.2mm_M2_ISO7380, F.Cu at (151.9, 53.3)
- added REF**: MountingHole_2.2mm_M2_ISO7380, MountingHole:MountingHole_2.2mm_M2_ISO7380, F.Cu at (60.0, 61.6)
- added REF**: MountingHole_2.2mm_M2_ISO7380, MountingHole:MountingHole_2.2mm_M2_ISO7380, F.Cu at (179.7, 117.5)
- D1, D10, D11, D12, D13, D14, D15, D17, D18, D19, D2, D20, D3, D4, D5, D6, D7, D8, D9: footprint keebio:Diode-dual -> keebio-parts:Diode-dual
- K1, K10, K11, K12, K13, K14, K15, K16, K17, K18, K2, K3, K4, K5, K6, K7, K8, K9: footprint project_footprints:SW_MX_reversible_minimal -> keyswitches:Kailh_socket_MX_optional_reversible
- moved J_2_RIGHT1 6.12 mm to (166.6, 93.2)
- moved J_1_LEFT1 6.12 mm to (166.6, 105.9)
- moved D11 3.82 mm to (79.1, 85.3)
- moved D13 2.31 mm to (79.1, 66.6)
- moved D8 1.42 mm to (98.1, 75.6)
- moved D18 1.29 mm to (140.2, 112.5)
- moved D17 1.23 mm to (163.2, 114.2)
- moved D19 1.04 mm to (155.6, 80.6)
- moved D5 0.95 mm to (117.3, 73.9)
- moved D20 0.84 mm to (155.4, 67.8)
- moved D1 0.82 mm to (136.2, 60.6)
- moved D4 0.77 mm to (117.2, 58.3)
- moved D2 0.75 mm to (136.2, 78.4)
- moved D6 0.71 mm to (117.2, 93.1)
- moved D7 0.66 mm to (98.2, 58.4)
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Routing:
- net GND: track 76.3 -> 2.51 mm, vias 0 -> 5
- net COL_2: track 221.3 -> 254.7 mm, vias 3 -> 12
- net REMOTE_COL_2: track 39.1 -> 69.2 mm, vias 0 -> 2
- net COL_1: track 171.7 -> 198.1 mm, vias 1 -> 6
- net REMOTE_COL_1: track 44.3 -> 67.3 mm, vias 0 -> 1
- net ROW_3: track 151.3 -> 171.4 mm, vias 0 -> 1
- net COL_3: track 288.1 -> 304.6 mm, vias 1 -> 6
- net ROW_2: track 164.6 -> 181.0 mm, vias 1 -> 2
- net ROW_4: track 90.3 -> 106.2 mm, vias 0 -> 1
- net Net-(D13-K): track 9.40 -> 25.3 mm, vias 0 -> 1
- net Net-(D7-K): track 20.2 -> 36.0 mm, vias 0 -> 1
- net Net-(D15-K): track 9.76 -> 25.5 mm, vias 0 -> 1
- net Net-(D18-A): track 7.10 -> 22.4 mm, vias 0 -> 1
- net Net-(D17-A): track 7.45 -> 22.3 mm, vias 0 -> 1
- net Net-(D5-A): track 23.4 -> 37.9 mm, vias 0 -> 3
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